Commit message: Add SROI gripper mesh and gripper_link to Piper URDF
Co-Authored-By: Claude Opus 4.7 <noreply@anthropic.com>

File: src/utils/piper_urdf/piper.urdf (robot description, URDF)
Before this commit: robot piper, 10 links, 9 joints
Links:
- added link gripper_link; collision mesh filename=meshes/sroi-piper-gripper.stl scale=0.001 0.001 0.001; visual mesh filename=meshes/sroi-piper-gripper.stl scale=0.001 0.001 0.001
Joints:
- added joint gripper_joint: type fixed, parent link6, child gripper_link, origin xyz=0 0 0 rpy=0 0 0
- joint camera_joint: origin xyz=-0.054333 0.00895 0.013471 rpy=-0.640492 0 -1.570797 -> xyz=-0.072333 0.00895 0.058471 rpy=-0.640492 0 -1.570797
- joint ee_joint: origin xyz=0 0 0.116517 rpy=0 0 -1.5707963 -> xyz=0 0 0.161517 rpy=0 0 -1.5707963
