Commit message: Add camera optical link and joint to gripper URDF

File: src/utils/piper_urdf/piper.urdf (robot description, URDF)
Before this commit: robot piper, 11 links, 10 joints
Links:
- added link camera_optical_link
Joints:
- added joint camera_optical_joint: type fixed, parent camera_link, child camera_optical_link, origin xyz=0 0 0 rpy=-1.5707963 0 -1.5707963
- joint camera_joint: origin xyz=-0.072333 0.00895 0.058471 rpy=-0.640492 0 -1.570797 -> xyz=-0.072333 0.00895 0.058471 rpy=0 -0.9303043 0
