Commit message: Update SROI Gripper URDF: refine comments, adjust origins, and replace mesh file

File: src/utils/piper_urdf/piper_sroiv2.urdf (robot description, URDF)
Before this commit: robot piper, 12 links, 11 joints
Links:
- link gripper_link: geometry collision mesh filename=meshes/sroiv2-piper-gripper.stl scale=1 1 1; visual mesh filename=meshes/sroiv2-piper-gripper.stl scale=1 1 1
Joints:
- joint gripper_joint: origin xyz=0 0 0 rpy=0 0 0 -> xyz=0 0 0 rpy=0 -1.5707963 0
